Commit message: .

File: urdf/quadcopter.xacro (robot description, xacro)
@@ -1,8 +1,8 @@
 <?xml version="1.0" ?>
 <robot name="quadcopter" xmlns:xacro="http://www.ros.org/wiki/xacro">
-<xacro:include filename="$(find quadcopter_description)/urdf/materials.xacro" />
-<xacro:include filename="$(find quadcopter_description)/urdf/quadcopter.trans" />
-<xacro:include filename="$(find quadcopter_description)/urdf/quadcopter.gazebo" />
-<xacro:include filename="$(find quadcopter_description)/urdf/quadmotor.xacro" />
+<xacro:include filename="$(find quadcopter_ros)/urdf/materials.xacro" />
+<xacro:include filename="$(find quadcopter_ros)/urdf/quadcopter.trans" />
+<xacro:include filename="$(find quadcopter_ros)/urdf/quadcopter.gazebo" />
+<xacro:include filename="$(find quadcopter_ros)/urdf/quadmotor.xacro" />
   <!-- making cylinder body approximation-->
   <!-- Inertia constants {-->
@@ -30,5 +30,5 @@
     <origin xyz="0 0 0" rpy="0 0 0"/>
     <geometry>
-      <mesh filename="package://quadcopter_description/meshes/base_link.stl" scale="0.001 0.001 0.001"/>
+      <mesh filename="package://quadcopter_ros/meshes/base_link.stl" scale="0.001 0.001 0.001"/>
     </geometry>
     <material name="plastic_glossy_grey"/>
@@ -37,5 +37,5 @@
     <origin xyz="0 0 0" rpy="0 0 0"/>
     <geometry>
-      <mesh filename="package://quadcopter_description/meshes/base_link.stl" scale="0.001 0.001 0.001"/>
+      <mesh filename="package://quadcopter_ros/meshes/base_link.stl" scale="0.001 0.001 0.001"/>
     </geometry>
   </collision>
@@ -50,5 +50,5 @@
     <origin xyz="-0.076368 0.099475 -0.03342" rpy="0 0 0"/>
     <geometry>
-      <mesh filename="package://quadcopter_description/meshes/prop1_1.stl" scale="0.001 0.001 0.001"/>
+      <mesh filename="package://quadcopter_ros/meshes/prop1_1.stl" scale="0.001 0.001 0.001"/>
     </geometry>
     <material name="abs_white"/>
@@ -57,5 +57,5 @@
     <origin xyz="-0.076368 0.099475 -0.03342" rpy="0 0 0"/>
     <geometry>
-      <mesh filename="package://quadcopter_description/meshes/prop1_1.stl" scale="0.001 0.001 0.001"/>
+      <mesh filename="package://quadcopter_ros/meshes/prop1_1.stl" scale="0.001 0.001 0.001"/>
     </geometry>
   </collision>
@@ -70,5 +70,5 @@
     <origin xyz="0.077777 0.099475 -0.03342" rpy="0 0 0"/>
     <geometry>
-      <mesh filename="package://quadcopter_description/meshes/prop2_1.stl" scale="0.001 0.001 0.001"/>
+      <mesh filename="package://quadcopter_ros/meshes/prop2_1.stl" scale="0.001 0.001 0.001"/>
     </geometry>
     <material name="abs_white"/>
@@ -77,5 +77,5 @@
     <origin xyz="0.077777 0.099475 -0.03342" rpy="0 0 0"/>
     <geometry>
-      <mesh filename="package://quadcopter_description/meshes/prop2_1.stl" scale="0.001 0.001 0.001"/>
+      <mesh filename="package://quadcopter_ros/meshes/prop2_1.stl" scale="0.001 0.001 0.001"/>
     </geometry>
   </collision>
@@ -90,5 +90,5 @@
     <origin xyz="0.077777 -0.099475 -0.03342" rpy="0 0 0"/>
     <geometry>
-      <mesh filename="package://quadcopter_description/meshes/prop3_1.stl" scale="0.001 0.001 0.001"/>
+      <mesh filename="package://quadcopter_ros/meshes/prop3_1.stl" scale="0.001 0.001 0.001"/>
     </geometry>
     <material name="abs_white"/>
@@ -97,5 +97,5 @@
     <origin xyz="0.077777 -0.099475 -0.03342" rpy="0 0 0"/>
     <geometry>
-      <mesh filename="package://quadcopter_description/meshes/prop3_1.stl" scale="0.001 0.001 0.001"/>
+      <mesh filename="package://quadcopter_ros/meshes/prop3_1.stl" scale="0.001 0.001 0.001"/>
     </geometry>
   </collision>
@@ -110,5 +110,5 @@
     <origin xyz="-0.076368 -0.099474 -0.03342" rpy="0 0 0"/>
     <geometry>
-      <mesh filename="package://quadcopter_description/meshes/prop4_1.stl" scale="0.001 0.001 0.001"/>
+      <mesh filename="package://quadcopter_ros/meshes/prop4_1.stl" scale="0.001 0.001 0.001"/>
     </geometry>
     <material name="abs_white"/>
@@ -117,5 +117,5 @@
     <origin xyz="-0.076368 -0.099474 -0.03342" rpy="0 0 0"/>
     <geometry>
-      <mesh filename="package://quadcopter_description/meshes/prop4_1.stl" scale="0.001 0.001 0.001"/>
+      <mesh filename="package://quadcopter_ros/meshes/prop4_1.stl" scale="0.001 0.001 0.001"/>
     </geometry>
   </collision>
